Commit message: update

File: src/x3cator_hardware/x3cator_model/urdf/x3cator_model.urdf (robot description, URDF)
Before this commit: robot x3cator_model, 1 links, 0 joints
Links:
- added link left_wheel, mass 2.0; collision cylinder length=0.05 radius=0.1; visual cylinder length=0.05 radius=0.1
- added link right_wheel, mass 2.0; collision cylinder length=0.05 radius=0.1; visual cylinder length=0.05 radius=0.1
- link base_link: mass 114.248 -> 20.0; geometry collision box size=0.5 0.3 0.2; visual mesh filename=package://x3cator_model/meshes/base_link.STL
Joints:
- added joint left_wheel_joint: type continuous, parent base_link, child left_wheel, origin xyz=0.0 0.4 -0.212 rpy=0 0 0, axis 0 1 0
- added joint right_wheel_joint: type continuous, parent base_link, child right_wheel, origin xyz=0.0 -0.4 -0.212 rpy=0 0 0, axis 0 1 0

Commit message: gazebo

File: src/x3cator_hardware/x3cator_model/urdf/x3cator_model.urdf (robot description, URDF)
Before this commit: robot x3cator_model, 3 links, 2 joints
Links:
- removed link left_wheel
- removed link right_wheel
- link base_link: mass 20.0 -> 114.248; geometry collision mesh filename=package://x3cator_model/meshes/base_link.STL; visual mesh filename=package://x3cator_model/meshes/base_link.STL
Joints:
- removed joint left_wheel_joint
- removed joint right_wheel_joint
