Commit message: urdf

File: src/x3cator_hardware/x3cator_model/urdf/x3cator_model_gazebo.urdf (robot description, URDF)
Before this commit: robot x3cator_model, 5 links, 4 joints
Links:
- added link imu_link, mass 0.1; collision box size=0.0 0.0 0.0; visual box size=0.0 0.0 0.0
- link camera_link: geometry collision box size=0.0 0.0 0.0; visual box size=0.0 0.0 0.0
- link lidar_link: geometry collision cylinder length=0.0 radius=0.0; visual cylinder length=0.0 radius=0.0
Joints:
- added joint imu_joint: type fixed, parent base_link, child imu_link, origin xyz=0.0 0.0 0.23 rpy=0 0 0
- joint camera_joint: origin xyz=0.53 0.0 0.13 rpy=0 0 0 -> xyz=0.53 0.0 0.23 rpy=0 0 0
- joint left_wheel_joint: origin xyz=0.0 0.35 -0.56 rpy=0 0 0 -> xyz=0.0 0.35 -0.26 rpy=0 0 0
- joint lidar_joint: origin xyz=0.437 0 0.429 rpy=0 0 0 -> xyz=0.437 0 0.45 rpy=0 0 0
- joint right_wheel_joint: origin xyz=0.0 -0.35 -0.56 rpy=0 0 0 -> xyz=0.0 -0.35 -0.26 rpy=0 0 0
